Commit message: FIX: collider

File: data/miku/urdf/miku.urdf (robot description, URDF)
Before this commit: robot miku, 75 links, 74 joints
Links:
- link left_foot: geometry collision box size=0.063 0.185 0.03; visual mesh filename=../meshes/left_foot_visual.stl
- link right_foot: geometry collision box size=0.063 0.185 0.03; visual mesh filename=../meshes/right_foot_visual.stl
