Commit message: UPDATE: model

File: data/miku/urdf/miku.urdf (robot description, URDF)
Before this commit: robot miku, 75 links, 74 joints
Links:
- removed link left_finger_1_distal
- removed link left_finger_1_intermediate
- removed link left_finger_1_mcp
- removed link left_finger_1_proximal
- removed link left_finger_2_distal
- removed link left_finger_2_intermediate
- removed link left_finger_2_mcp
- removed link left_finger_2_proximal
- removed link left_finger_3_distal
- removed link left_finger_3_intermediate
- removed link left_finger_3_mcp
- removed link left_finger_3_proximal
- removed link left_finger_4_distal
- removed link left_finger_4_intermediate
- removed link left_finger_4_mcp
- removed link left_finger_4_proximal
- removed link left_finger_5_distal
- removed link left_finger_5_intermediate
- removed link left_finger_5_mcp
- removed link left_finger_5_proximal
- removed link left_palm
- removed link right_finger_1_distal
- removed link right_finger_1_intermediate
- removed link right_finger_1_mcp
- removed link right_finger_1_proximal
- removed link right_finger_2_distal
- removed link right_finger_2_intermediate
- removed link right_finger_2_mcp
- removed link right_finger_2_proximal
- removed link right_finger_3_distal
- removed link right_finger_3_intermediate
- removed link right_finger_3_mcp
- removed link right_finger_3_proximal
- removed link right_finger_4_distal
- removed link right_finger_4_intermediate
- removed link right_finger_4_mcp
- removed link right_finger_4_proximal
- removed link right_finger_5_distal
- removed link right_finger_5_intermediate
- removed link right_finger_5_mcp
- removed link right_finger_5_proximal
- removed link right_palm
- removed link shoulder_base
- added link left_finger_1_j1, mass 0.000744; visual mesh filename=../meshes/left_finger_1_j1_visual.stl
- added link left_finger_1_j2, mass 0.002976; visual mesh filename=../meshes/left_finger_1_j2_visual.stl
- added link left_finger_1_j3, mass 0.001984; visual mesh filename=../meshes/left_finger_1_j3_visual.stl
- added link left_finger_1_j4, mass 0.001333; visual mesh filename=../meshes/left_finger_1_j4_visual.stl
- added link left_finger_2_j1, mass 0.000496; visual mesh filename=../meshes/left_finger_2_j1_visual.stl
- added link left_finger_2_j2, mass 0.00248; visual mesh filename=../meshes/left_finger_2_j2_visual.stl
- added link left_finger_2_j3, mass 0.0011904; visual mesh filename=../meshes/left_finger_2_j3_visual.stl
- added link left_finger_2_j4, mass 0.0004185; visual mesh filename=../meshes/left_finger_2_j4_visual.stl
- added link left_finger_3_j1, mass 0.000496; visual mesh filename=../meshes/left_finger_3_j1_visual.stl
- added link left_finger_3_j2, mass 0.002976; visual mesh filename=../meshes/left_finger_3_j2_visual.stl
- added link left_finger_3_j3, mass 0.001488; visual mesh filename=../meshes/left_finger_3_j3_visual.stl
- added link left_finger_3_j4, mass 0.0004185; visual mesh filename=../meshes/left_finger_3_j4_visual.stl
- added link left_finger_4_j1, mass 0.000496; visual mesh filename=../meshes/left_finger_4_j1_visual.stl
- added link left_finger_4_j2, mass 0.002976; visual mesh filename=../meshes/left_finger_4_j2_visual.stl
- added link left_finger_4_j3, mass 0.0011904; visual mesh filename=../meshes/left_finger_4_j3_visual.stl
- added link left_finger_4_j4, mass 0.0004185; visual mesh filename=../meshes/left_finger_4_j4_visual.stl
- added link left_finger_5_j1, mass 0.000496; visual mesh filename=../meshes/left_finger_5_j1_visual.stl
- added link left_finger_5_j2, mass 0.001984; visual mesh filename=../meshes/left_finger_5_j2_visual.stl
- added link left_finger_5_j3, mass 0.0008928; visual mesh filename=../meshes/left_finger_5_j3_visual.stl
- added link left_finger_5_j4, mass 0.0004185; visual mesh filename=../meshes/left_finger_5_j4_visual.stl
- added link left_hand, mass 0.028365; collision box size=0.1 0.07 0.015; visual mesh filename=../meshes/left_hand_visual.stl
- added link right_finger_1_j1, mass 0.000744; visual mesh filename=../meshes/right_finger_1_j1_visual.stl
- added link right_finger_1_j2, mass 0.002976; visual mesh filename=../meshes/right_finger_1_j2_visual.stl
- added link right_finger_1_j3, mass 0.001984; visual mesh filename=../meshes/right_finger_1_j3_visual.stl
- added link right_finger_1_j4, mass 0.001333; visual mesh filename=../meshes/right_finger_1_j4_visual.stl
- added link right_finger_2_j1, mass 0.000496; visual mesh filename=../meshes/right_finger_2_j1_visual.stl
- added link right_finger_2_j2, mass 0.00248; visual mesh filename=../meshes/right_finger_2_j2_visual.stl
- added link right_finger_2_j3, mass 0.0011904; visual mesh filename=../meshes/right_finger_2_j3_visual.stl
- added link right_finger_2_j4, mass 0.0004185; visual mesh filename=../meshes/right_finger_2_j4_visual.stl
- added link right_finger_3_j1, mass 0.000496; visual mesh filename=../meshes/right_finger_3_j1_visual.stl
- added link right_finger_3_j2, mass 0.002976; visual mesh filename=../meshes/right_finger_3_j2_visual.stl
- added link right_finger_3_j3, mass 0.001488; visual mesh filename=../meshes/right_finger_3_j3_visual.stl
- added link right_finger_3_j4, mass 0.0004185; visual mesh filename=../meshes/right_finger_3_j4_visual.stl
- added link right_finger_4_j1, mass 0.000496; visual mesh filename=../meshes/right_finger_4_j1_visual.stl
- added link right_finger_4_j2, mass 0.002976; visual mesh filename=../meshes/right_finger_4_j2_visual.stl
- added link right_finger_4_j3, mass 0.0011904; visual mesh filename=../meshes/right_finger_4_j3_visual.stl
- added link right_finger_4_j4, mass 0.0004185; visual mesh filename=../meshes/right_finger_4_j4_visual.stl
- added link right_finger_5_j1, mass 0.000496; visual mesh filename=../meshes/right_finger_5_j1_visual.stl
- added link right_finger_5_j2, mass 0.001984; visual mesh filename=../meshes/right_finger_5_j2_visual.stl
- added link right_finger_5_j3, mass 0.0008928; visual mesh filename=../meshes/right_finger_5_j3_visual.stl
- added link right_finger_5_j4, mass 0.0004185; visual mesh filename=../meshes/right_finger_5_j4_visual.stl
- added link right_hand, mass 0.028365; collision box size=0.1 0.07 0.015; visual mesh filename=../meshes/right_hand_visual.stl
- added link torso, mass 1.31699; collision cylinder length=0.08 radius=0.05; collision cylinder length=0.12 radius=0.04
- link head: mass 4.73312 -> 4.83041; geometry collision cylinder length=0.03 radius=0.09; visual mesh filename=../meshes/head_visual.stl
- link left_knee_pitch: mass 2.86325 -> 2.92168; geometry collision cylinder length=0.16 radius=0.05; visual mesh filename=../meshes/left_knee_pitch_visual.stl
- link left_shoulder_roll: mass 0.476818 -> 0.455782
- link pelvis: geometry collision cylinder length=0.1 radius=0.05; collision cylinder length=0.16 radius=0.05
- link right_knee_pitch: mass 2.86325 -> 2.92168; geometry collision cylinder length=0.16 radius=0.05; visual mesh filename=../meshes/right_knee_pitch_visual.stl
- link right_shoulder_roll: mass 0.476818 -> 0.455782
Joints:
- removed joint left_hand_finger1_joint1
- removed joint left_hand_finger1_joint2
- removed joint left_hand_finger1_joint3
- removed joint left_hand_finger1_joint4
- removed joint left_hand_finger2_joint1
- removed joint left_hand_finger2_joint2
- removed joint left_hand_finger2_joint3
- removed joint left_hand_finger2_joint4
- removed joint left_hand_finger3_joint1
- removed joint left_hand_finger3_joint2
- removed joint left_hand_finger3_joint3
- removed joint left_hand_finger3_joint4
- removed joint left_hand_finger4_joint1
- removed joint left_hand_finger4_joint2
- removed joint left_hand_finger4_joint3
- removed joint left_hand_finger4_joint4
- removed joint left_hand_finger5_joint1
- removed joint left_hand_finger5_joint2
- removed joint left_hand_finger5_joint3
- removed joint left_hand_finger5_joint4
- removed joint right_hand_finger1_joint1
- removed joint right_hand_finger1_joint2
- removed joint right_hand_finger1_joint3
- removed joint right_hand_finger1_joint4
- removed joint right_hand_finger2_joint1
- removed joint right_hand_finger2_joint2
- removed joint right_hand_finger2_joint3
- removed joint right_hand_finger2_joint4
- removed joint right_hand_finger3_joint1
- removed joint right_hand_finger3_joint2
- removed joint right_hand_finger3_joint3
- removed joint right_hand_finger3_joint4
- removed joint right_hand_finger4_joint1
- removed joint right_hand_finger4_joint2
- removed joint right_hand_finger4_joint3
- removed joint right_hand_finger4_joint4
- removed joint right_hand_finger5_joint1
- removed joint right_hand_finger5_joint2
- removed joint right_hand_finger5_joint3
- removed joint right_hand_finger5_joint4
- added joint left_finger1_j1: type revolute, parent left_hand, child left_finger_1_j1, origin xyz=0 0.035 0.015 rpy=0.785398 0 -0, axis 0 0 1, limit lower=-1.91986 upper=0.0872665 effort=100 velocity=100
- added joint left_finger1_j2: type revolute, parent left_finger_1_j1, child left_finger_1_j2, origin xyz=0 0.01 -0 rpy=0 -1.5708 0, axis 0 0 1, limit lower=-0.349066 upper=0.349066 effort=100 velocity=100
- added joint left_finger1_j3: type revolute, parent left_finger_1_j2, child left_finger_1_j3, origin xyz=0 0.025 0 rpy=0 1.5708 0, axis 0 0 1, limit lower=-1.91986 upper=0.0872665 effort=100 velocity=100
- added joint left_finger1_j4: type revolute, parent left_finger_1_j3, child left_finger_1_j4, origin xyz=0 0.025 0 rpy=-0 0 -0, axis 0 0 1, limit lower=-1.91986 upper=0.0872665 effort=100 velocity=100
- added joint left_finger2_j1: type revolute, parent left_hand, child left_finger_2_j1, origin xyz=0 0.07 0.015 rpy=-0 0 -0, axis 0 0 1, limit lower=-1.91986 upper=0.0872665 effort=100 velocity=100
- added joint left_finger2_j2: type revolute, parent left_finger_2_j1, child left_finger_2_j2, origin xyz=0 0.01 0 rpy=0 -1.5708 0, axis 0 0 1, limit lower=-0.349066 upper=0.349066 effort=100 velocity=100
- added joint left_finger2_j3: type revolute, parent left_finger_2_j2, child left_finger_2_j3, origin xyz=-0 0.03 0 rpy=0 1.5708 0, axis 0 0 1, limit lower=-1.91986 upper=0.0872665 effort=100 velocity=100
- added joint left_finger2_j4: type revolute, parent left_finger_2_j3, child left_finger_2_j4, origin xyz=0 0.025 0 rpy=0 0 -0, axis 0 0 1, limit lower=-1.91986 upper=0.0872665 effort=100 velocity=100
- added joint left_finger3_j1: type revolute, parent left_hand, child left_finger_3_j1, origin xyz=0 0.07 0 rpy=-0 0 -0, axis 0 0 1, limit lower=-1.91986 upper=0.0872665 effort=100 velocity=100
- added joint left_finger3_j2: type revolute, parent left_finger_3_j1, child left_finger_3_j2, origin xyz=0 0.01 -0 rpy=-0 -1.5708 0, axis 0 0 1, limit lower=-0.349066 upper=0.349066 effort=100 velocity=100
- added joint left_finger3_j3: type revolute, parent left_finger_3_j2, child left_finger_3_j3, origin xyz=0 0.035 0 rpy=-0 1.5708 0, axis 0 0 1, limit lower=-1.91986 upper=0.0872665 effort=100 velocity=100
- added joint left_finger3_j4: type revolute, parent left_finger_3_j3, child left_finger_3_j4, origin xyz=0 0.03 0 rpy=-0 0 0, axis 0 0 1, limit lower=-1.91986 upper=0.0872665 effort=100 velocity=100
- added joint left_finger4_j1: type revolute, parent left_hand, child left_finger_4_j1, origin xyz=0 0.07 -0.015 rpy=-0 0 -0, axis 0 0 1, limit lower=-1.91986 upper=0.0872665 effort=100 velocity=100
- added joint left_finger4_j2: type revolute, parent left_finger_4_j1, child left_finger_4_j2, origin xyz=0 0.01 0 rpy=0 -1.5708 0, axis 0 0 1, limit lower=-0.349066 upper=0.349066 effort=100 velocity=100
- added joint left_finger4_j3: type revolute, parent left_finger_4_j2, child left_finger_4_j3, origin xyz=-0 0.035 0 rpy=0 1.5708 0, axis 0 0 1, limit lower=-1.91986 upper=0.0872665 effort=100 velocity=100
- added joint left_finger4_j4: type revolute, parent left_finger_4_j3, child left_finger_4_j4, origin xyz=-0 0.025 0 rpy=0 -0 0, axis 0 0 1, limit lower=-1.91986 upper=0.0872665 effort=100 velocity=100
- added joint left_finger5_j1: type revolute, parent left_hand, child left_finger_5_j1, origin xyz=0 0.07 -0.03 rpy=-0 0 -0, axis 0 0 1, limit lower=-1.91986 upper=0.0872665 effort=100 velocity=100
- added joint left_finger5_j2: type revolute, parent left_finger_5_j1, child left_finger_5_j2, origin xyz=0 0.01 -0 rpy=0 -1.5708 0, axis 0 0 1, limit lower=-0.349066 upper=0.349066 effort=100 velocity=100
- added joint left_finger5_j3: type revolute, parent left_finger_5_j2, child left_finger_5_j3, origin xyz=0 0.025 0 rpy=0 1.5708 0, axis 0 0 1, limit lower=-1.91986 upper=0.0872665 effort=100 velocity=100
- added joint left_finger5_j4: type revolute, parent left_finger_5_j3, child left_finger_5_j4, origin xyz=-0 0.02 0 rpy=-0 0 -0, axis 0 0 1, limit lower=-1.91986 upper=0.0872665 effort=100 velocity=100
- added joint right_finger1_j1: type revolute, parent right_hand, child right_finger_1_j1, origin xyz=0 0.035 0.015 rpy=0.785398 0 0, axis 0 0 1, limit lower=-0.0872665 upper=1.91986 effort=100 velocity=100
- added joint right_finger1_j2: type revolute, parent right_finger_1_j1, child right_finger_1_j2, origin xyz=-0 0.01 -0 rpy=0 1.5708 0, axis 0 0 1, limit lower=-0.349066 upper=0.349066 effort=100 velocity=100
- added joint right_finger1_j3: type revolute, parent right_finger_1_j2, child right_finger_1_j3, origin xyz=0 0.025 0 rpy=-0 -1.5708 0, axis 0 0 1, limit lower=-0.0872665 upper=1.91986 effort=100 velocity=100
- added joint right_finger1_j4: type revolute, parent right_finger_1_j3, child right_finger_1_j4, origin xyz=0 0.025 -0 rpy=-0 0 -0, axis 0 0 1, limit lower=-0.0872665 upper=1.91986 effort=100 velocity=100
- added joint right_finger2_j1: type revolute, parent right_hand, child right_finger_2_j1, origin xyz=0 0.07 0.015 rpy=0 0 0, axis 0 0 1, limit lower=-0.0872665 upper=1.91986 effort=100 velocity=100
- added joint right_finger2_j2: type revolute, parent right_finger_2_j1, child right_finger_2_j2, origin xyz=-0 0.01 -0 rpy=0 1.5708 0, axis 0 0 1, limit lower=-0.349066 upper=0.349066 effort=100 velocity=100
- added joint right_finger2_j3: type revolute, parent right_finger_2_j2, child right_finger_2_j3, origin xyz=0 0.03 0 rpy=0 -1.5708 0, axis 0 0 1, limit lower=-0.0872665 upper=1.91986 effort=100 velocity=100
- added joint right_finger2_j4: type revolute, parent right_finger_2_j3, child right_finger_2_j4, origin xyz=0 0.025 -0 rpy=0 0 0, axis 0 0 1, limit lower=-0.0872665 upper=1.91986 effort=100 velocity=100
- added joint right_finger3_j1: type revolute, parent right_hand, child right_finger_3_j1, origin xyz=0 0.07 -0 rpy=0 0 -0, axis 0 0 1, limit lower=-0.0872665 upper=1.91986 effort=100 velocity=100
- added joint right_finger3_j2: type revolute, parent right_finger_3_j1, child right_finger_3_j2, origin xyz=0 0.01 0 rpy=-0 1.5708 0, axis 0 0 1, limit lower=-0.349066 upper=0.349066 effort=100 velocity=100
- added joint right_finger3_j3: type revolute, parent right_finger_3_j2, child right_finger_3_j3, origin xyz=0 0.035 0 rpy=0 -1.5708 0, axis 0 0 1, limit lower=-0.0872665 upper=1.91986 effort=100 velocity=100
- added joint right_finger3_j4: type revolute, parent right_finger_3_j3, child right_finger_3_j4, origin xyz=-0 0.03 -0 rpy=0 0 0, axis 0 0 1, limit lower=-0.0872665 upper=1.91986 effort=100 velocity=100
- added joint right_finger4_j1: type revolute, parent right_hand, child right_finger_4_j1, origin xyz=0 0.07 -0.015 rpy=-0 0 -0, axis 0 0 1, limit lower=-0.0872665 upper=1.91986 effort=100 velocity=100
- added joint right_finger4_j2: type revolute, parent right_finger_4_j1, child right_finger_4_j2, origin xyz=0 0.01 0 rpy=-0 1.5708 0, axis 0 0 1, limit lower=-0.349066 upper=0.349066 effort=100 velocity=100
- added joint right_finger4_j3: type revolute, parent right_finger_4_j2, child right_finger_4_j3, origin xyz=0 0.035 -0 rpy=-0 -1.5708 0, axis 0 0 1, limit lower=-0.0872665 upper=1.91986 effort=100 velocity=100
- added joint right_finger4_j4: type revolute, parent right_finger_4_j3, child right_finger_4_j4, origin xyz=0 0.025 0 rpy=-0 0 0, axis 0 0 1, limit lower=-0.0872665 upper=1.91986 effort=100 velocity=100
- added joint right_finger5_j1: type revolute, parent right_hand, child right_finger_5_j1, origin xyz=0 0.07 -0.03 rpy=0 0 -0, axis 0 0 1, limit lower=-0.0872665 upper=1.91986 effort=100 velocity=100
- added joint right_finger5_j2: type revolute, parent right_finger_5_j1, child right_finger_5_j2, origin xyz=0 0.01 -0 rpy=-0 1.5708 0, axis 0 0 1, limit lower=-0.349066 upper=0.349066 effort=100 velocity=100
- added joint right_finger5_j3: type revolute, parent right_finger_5_j2, child right_finger_5_j3, origin xyz=0 0.025 -0 rpy=-0 -1.5708 0, axis 0 0 1, limit lower=-0.0872665 upper=1.91986 effort=100 velocity=100
- added joint right_finger5_j4: type revolute, parent right_finger_5_j3, child right_finger_5_j4, origin xyz=-0 0.02 0 rpy=0 0 0, axis 0 0 1, limit lower=-0.0872665 upper=1.91986 effort=100 velocity=100
- joint left_ankle_pitch: child right_foot -> left_foot; origin xyz=0.025 0 -0.025 rpy=1.08468e-29 1.5708 0 -> xyz=0 -0 0 rpy=0 -1.5708 0; parent right_ankle_yaw -> left_ankle_roll
- joint left_ankle_roll: child right_ankle_yaw -> left_ankle_roll; origin xyz=4.16334e-17 0.025 0.05 rpy=-1.5708 9.26912e-30 6.52656e-28 -> xyz=0 0 0 rpy=-1.5708 -0 -1.5708; parent right_ankle_roll -> left_ankle_yaw
- joint left_ankle_yaw: child right_ankle_roll -> left_ankle_yaw; origin xyz=1.00005e-17 -0.344 -0.025 rpy=1.5708 -1.5708 0 -> xyz=0 0.4 0 rpy=1.5708 0 0; parent right_knee_pitch -> left_knee_pitch
- joint left_elbow_pitch: origin xyz=1.83697e-18 -0.025 0.03 rpy=1.5708 1.5708 0 -> xyz=0 -0 0.2 rpy=1.5708 0 -0
- joint left_hip_pitch: child right_hip_pitch -> left_hip_pitch; limit lower=-0.785398 upper=2.35619 effort=100 velocity=100 -> lower=-2.35619 upper=0.785398 effort=100 velocity=100; origin xyz=-3.06162e-18 -0.08 0.89 rpy=1.5708 2.10942e-15 -7.12835e-15 -> xyz=-0 0.08 0 rpy=-1.5708 -0 0
- joint left_hip_roll: child right_hip_roll -> left_hip_roll; origin xyz=-0.05 -1.11022e-16 -1.38778e-17 rpy=-3.14159 -1.5708 0 -> xyz=0 -0 -0 rpy=0 1.5708 0; parent right_hip_pitch -> left_hip_pitch
- joint left_hip_yaw: child right_hip_yaw -> left_hip_yaw; origin xyz=0 0.37 0.05 rpy=-1.5708 1.249e-15 -2.77556e-17 -> xyz=0 0 -0 rpy=1.5708 -1.5708 0; parent right_hip_roll -> left_hip_roll
- joint left_knee_pitch: child right_knee_pitch -> left_knee_pitch; limit lower=-2.35619 upper=3.55271e-15 effort=100 velocity=100 -> lower=0 upper=2.35619 effort=100 velocity=100; origin xyz=0.025 3.06162e-18 0.05 rpy=-1.5708 3.01986e-30 -1.5708 -> xyz=-0 0 -0.42 rpy=-1.5708 -0 -0; parent right_hip_yaw -> left_hip_yaw
- joint left_shoulder_pitch: origin xyz=-0.052 -0.16948 -0.025 rpy=2.52353e-32 -1.5708 0 -> xyz=0.09 0.17 0 rpy=-3.14159 -1.5708 0; parent shoulder_base -> torso
- joint left_shoulder_roll: limit lower=-3.14159 upper=0.261799 effort=100 velocity=100 -> lower=-1.74533 upper=1.74533 effort=100 velocity=100; origin xyz=0.025 -2.22045e-16 0.04 rpy=3.69779e-31 1.5708 0 -> xyz=0 0 0 rpy=1.5708 -0 1.5708
- joint left_shoulder_yaw: origin xyz=-0.176 0 -0.025 rpy=-1.72563e-29 -1.5708 0 -> xyz=0 0 0 rpy=-1.5708 -1.5708 0
- joint left_wrist_pitch: child left_palm -> left_hand; origin xyz=-5.55112e-17 0.025 -0.025 rpy=-1.5708 -1.04761e-27 -5.55112e-17 -> xyz=-0 -0 0 rpy=0 1.5708 0; parent left_wrist_yaw -> left_wrist_roll
- joint left_wrist_roll: child left_wrist_yaw -> left_wrist_roll; origin xyz=1.34988e-18 -0.025 0.025 rpy=1.5708 1.5708 0 -> xyz=0 0 0 rpy=1.5708 0 -0; parent left_wrist_roll -> left_wrist_yaw
- joint left_wrist_yaw: child left_wrist_roll -> left_wrist_yaw; origin xyz=-0.155 -1.9622e-18 -0.025 rpy=-1.5708 7.88861e-31 1.5708 -> xyz=-0 0.18 0 rpy=-1.5708 0 0
- joint neck_pitch: origin xyz=0.025 -0.05 -0.035 rpy=3.14159 -1.5708 0 -> xyz=-0 0.04 0 rpy=-0 1.5708 0
- joint neck_roll: origin xyz=-9.70628e-19 0.025 0.03 rpy=-1.5708 -5.52203e-30 6.12323e-17 -> xyz=-0 0 0.04 rpy=1.5708 -0 1.5708
- joint neck_yaw: origin xyz=-1.72556e-18 -0.21948 -0.025 rpy=1.5708 3.31821e-30 1.56492e-15 -> xyz=-0 0.23 0 rpy=-1.5708 -1.5708 0; parent shoulder_base -> torso
- joint right_ankle_pitch: child left_foot -> right_foot; origin xyz=-0.025 0 -0.025 rpy=3.14159 1.5708 0 -> xyz=0 0 -0 rpy=-0 -1.5708 0; parent left_ankle_yaw -> right_ankle_roll
- joint right_ankle_roll: child left_ankle_yaw -> right_ankle_roll; origin xyz=-1.38778e-17 0.025 0.05 rpy=-1.5708 2.02825e-15 6.12323e-17 -> xyz=0 0 0 rpy=-1.5708 0 -1.5708; parent left_ankle_roll -> right_ankle_yaw
- joint right_ankle_yaw: child left_ankle_roll -> right_ankle_yaw; origin xyz=6.29306e-15 0.344 -0.025 rpy=-1.5708 1.5708 0 -> xyz=0 0.4 0 rpy=1.5708 -0 0; parent left_knee_pitch -> right_knee_pitch
- joint right_elbow_pitch: limit lower=-0 upper=2.35619 effort=100 velocity=100 -> lower=-2.35619 upper=0 effort=100 velocity=100; origin xyz=8.23975e-16 0.025 0.03 rpy=-1.5708 -1.5708 0 -> xyz=-0 -0 0.2 rpy=1.5708 -0 -0
- joint right_hip_pitch: child left_hip_pitch -> right_hip_pitch; origin xyz=-3.06162e-18 0.08 0.89 rpy=-1.5708 -1.57772e-30 1.44329e-15 -> xyz=0 -0.08 0 rpy=-1.5708 0 0
- joint right_hip_roll: child left_hip_roll -> right_hip_roll; origin xyz=-0.05 0 0 rpy=-3.51538e-16 1.5708 0 -> xyz=-0 -0 0 rpy=0 1.5708 0; parent left_hip_pitch -> right_hip_pitch
- joint right_hip_yaw: child left_hip_yaw -> right_hip_yaw; origin xyz=0 0.37 0.05 rpy=-1.5708 9.99201e-16 -1.906e-15 -> xyz=0 0 0 rpy=1.5708 -1.5708 0; parent left_hip_roll -> right_hip_roll
- joint right_knee_pitch: child left_knee_pitch -> right_knee_pitch; limit lower=-0 upper=2.35619 effort=100 velocity=100 -> lower=0 upper=2.35619 effort=100 velocity=100; origin xyz=-0.025 3.06162e-18 0.05 rpy=1.5708 2.66241e-30 -1.5708 -> xyz=-0 -0 -0.42 rpy=-1.5708 0 0; parent left_hip_yaw -> right_hip_yaw
- joint right_shoulder_pitch: origin xyz=0.052 -0.16948 -0.025 rpy=3.14159 -1.5708 0 -> xyz=-0.09 0.17 -0 rpy=-3.14159 -1.5708 0; parent shoulder_base -> torso
- joint right_shoulder_roll: limit lower=-0.261799 upper=3.14159 effort=100 velocity=100 -> lower=-1.74533 upper=1.74533 effort=100 velocity=100; origin xyz=0.025 -3.10862e-15 0.04 rpy=-3.14159 -1.5708 0 -> xyz=-0 0 0 rpy=1.5708 -0 1.5708
- joint right_shoulder_yaw: origin xyz=0.176 -2.22045e-16 -0.025 rpy=-3.14159 -1.5708 0 -> xyz=0 0 0 rpy=1.5708 -1.5708 0
- joint right_wrist_pitch: child right_palm -> right_hand; origin xyz=-2.9976e-15 0.025 -0.025 rpy=-1.5708 -1.69201e-15 5.41428e-30 -> xyz=0 0 0 rpy=0 1.5708 0; parent right_wrist_yaw -> right_wrist_roll
- joint right_wrist_roll: child right_wrist_yaw -> right_wrist_roll; origin xyz=1.22465e-18 0.025 0.025 rpy=-1.5708 -1.5708 0 -> xyz=-0 0 0 rpy=1.5708 0 0; parent right_wrist_roll -> right_wrist_yaw
- joint right_wrist_yaw: child right_wrist_roll -> right_wrist_yaw; origin xyz=0.155 1.78385e-18 -0.025 rpy=1.5708 8.19657e-16 1.5708 -> xyz=0 0.18 0 rpy=-1.5708 -0 -0
- joint waist_pitch: limit lower=-0.523599 upper=0.523599 effort=100 velocity=100 -> lower=-0.785398 upper=1.5708 effort=100 velocity=100; origin xyz=0.025 -6.91715e-18 0.040516 rpy=1.5708 -8.73285e-28 1.5708 -> xyz=0 -0 0 rpy=1.5708 0 3.14159
- joint waist_roll: child shoulder_base -> torso; limit lower=-0.523599 upper=0.523599 effort=100 velocity=100 -> lower=-1.0472 upper=1.0472 effort=100 velocity=100; origin xyz=0.025 0.118004 -0.025 rpy=-3.14159 -1.5708 0 -> xyz=-0 0.09 -0 rpy=0 -1.5708 0
- joint waist_yaw: limit lower=-0.785398 upper=0.785398 effort=100 velocity=100 -> lower=-1.5708 upper=1.5708 effort=100 velocity=100; origin xyz=0 0 0.94 rpy=-1.32608e-27 -2.58745e-28 -1.5708 -> xyz=0 -0 0.12 rpy=-0 -0 0
