Commit message: update: shoulder and hip tilt

File: data/miku/urdf/miku.urdf (robot description, URDF)
Before this commit: robot miku, 75 links, 74 joints
Links:
- link pelvis: mass 1.63184 -> 1.63182
- link torso: mass 1.31699 -> 1.30495
Joints:
- joint left_ankle_pitch: origin xyz=0 -0 0 rpy=0 -1.5708 0 -> xyz=0 0 0 rpy=-0 -1.5708 0
- joint left_ankle_yaw: origin xyz=0 0.4 0 rpy=1.5708 0 0 -> xyz=0 0.4 0 rpy=1.5708 -0 0
- joint left_elbow_pitch: origin xyz=0 -0 0.2 rpy=1.5708 0 -0 -> xyz=0 -0 0.2 rpy=1.5708 -0 -0
- joint left_finger1_j1: origin xyz=0 0.035 0.015 rpy=0.785398 0 -0 -> xyz=-0 0.035 0.015 rpy=0.785398 0 0
- joint left_finger1_j3: origin xyz=0 0.025 0 rpy=0 1.5708 0 -> xyz=-0 0.025 0 rpy=0 1.5708 0
- joint left_finger1_j4: origin xyz=0 0.025 0 rpy=-0 0 -0 -> xyz=0 0.025 0 rpy=0 -0 -0
- joint left_finger2_j1: origin xyz=0 0.07 0.015 rpy=-0 0 -0 -> xyz=-0 0.07 0.015 rpy=0 0 -0
- joint left_finger2_j2: origin xyz=0 0.01 0 rpy=0 -1.5708 0 -> xyz=-0 0.01 0 rpy=-0 -1.5708 0
- joint left_finger2_j3: origin xyz=-0 0.03 0 rpy=0 1.5708 0 -> xyz=0 0.03 0 rpy=-0 1.5708 0
- joint left_finger2_j4: origin xyz=0 0.025 0 rpy=0 0 -0 -> xyz=0 0.025 -0 rpy=0 0 -0
- joint left_finger3_j1: origin xyz=0 0.07 0 rpy=-0 0 -0 -> xyz=0 0.07 0 rpy=-0 0 0
- joint left_finger3_j2: origin xyz=0 0.01 -0 rpy=-0 -1.5708 0 -> xyz=0 0.01 0 rpy=0 -1.5708 0
- joint left_finger3_j4: origin xyz=0 0.03 0 rpy=-0 0 0 -> xyz=0 0.03 -0 rpy=0 0 -0
- joint left_finger4_j1: origin xyz=0 0.07 -0.015 rpy=-0 0 -0 -> xyz=0 0.07 -0.015 rpy=-0 0 0
- joint left_finger4_j3: origin xyz=-0 0.035 0 rpy=0 1.5708 0 -> xyz=0 0.035 0 rpy=0 1.5708 0
- joint left_finger4_j4: origin xyz=-0 0.025 0 rpy=0 -0 0 -> xyz=0 0.025 0 rpy=-0 0 0
- joint left_finger5_j1: origin xyz=0 0.07 -0.03 rpy=-0 0 -0 -> xyz=0 0.07 -0.03 rpy=0 0 0
- joint left_finger5_j2: origin xyz=0 0.01 -0 rpy=0 -1.5708 0 -> xyz=0 0.01 0 rpy=-0 -1.5708 0
- joint left_finger5_j3: origin xyz=0 0.025 0 rpy=0 1.5708 0 -> xyz=0 0.025 0 rpy=-0 1.5708 0
- joint left_finger5_j4: origin xyz=-0 0.02 0 rpy=-0 0 -0 -> xyz=0 0.02 0 rpy=-0 -0 0
- joint left_hip_pitch: origin xyz=-0 0.08 0 rpy=-1.5708 -0 0 -> xyz=1.36e-09 0.08 1.6286e-08 rpy=-1.74533 0 0
- joint left_hip_roll: origin xyz=0 -0 -0 rpy=0 1.5708 0 -> xyz=-0 0 -0 rpy=1.5708 1.39626 1.5708
- joint left_hip_yaw: origin xyz=0 0 -0 rpy=1.5708 -1.5708 0 -> xyz=-0 0 0 rpy=1.5708 -1.5708 0
- joint left_knee_pitch: origin xyz=-0 0 -0.42 rpy=-1.5708 -0 -0 -> xyz=-0 -0 -0.42 rpy=-1.5708 0 -0
- joint left_shoulder_pitch: origin xyz=0.09 0.17 0 rpy=-3.14159 -1.5708 0 -> xyz=0.0887752 0.176946 0 rpy=-2.96706 -1.5708 0
- joint left_shoulder_roll: limit lower=-1.74533 upper=1.74533 effort=100 velocity=100 -> lower=-0.174533 upper=3.14159 effort=100 velocity=100; origin xyz=0 0 0 rpy=1.5708 -0 1.5708 -> xyz=-0 0 0 rpy=1.5708 0.174533 1.5708
- joint left_wrist_pitch: origin xyz=-0 -0 0 rpy=0 1.5708 0 -> xyz=0 0 0 rpy=0 1.5708 0
- joint left_wrist_yaw: origin xyz=-0 0.18 0 rpy=-1.5708 0 0 -> xyz=0 0.18 -0 rpy=-1.5708 -0 0
- joint neck_pitch: origin xyz=-0 0.04 0 rpy=-0 1.5708 0 -> xyz=0 0.04 0 rpy=-0 1.5708 0
- joint neck_roll: origin xyz=-0 0 0.04 rpy=1.5708 -0 1.5708 -> xyz=-0 -0 0.04 rpy=1.5708 0 1.5708
- joint right_ankle_pitch: origin xyz=0 0 -0 rpy=-0 -1.5708 0 -> xyz=0 0 0 rpy=0 -1.5708 0
- joint right_ankle_yaw: origin xyz=0 0.4 0 rpy=1.5708 -0 0 -> xyz=0 0.4 0 rpy=1.5708 -0 -0
- joint right_elbow_pitch: origin xyz=-0 -0 0.2 rpy=1.5708 -0 -0 -> xyz=0 0 0.2 rpy=1.5708 0 -0
- joint right_finger1_j2: origin xyz=-0 0.01 -0 rpy=0 1.5708 0 -> xyz=0 0.01 -0 rpy=-0 1.5708 0
- joint right_finger1_j3: origin xyz=0 0.025 0 rpy=-0 -1.5708 0 -> xyz=-0 0.025 0 rpy=0 -1.5708 0
- joint right_finger1_j4: origin xyz=0 0.025 -0 rpy=-0 0 -0 -> xyz=0 0.025 0 rpy=-0 0 -0
- joint right_finger2_j1: origin xyz=0 0.07 0.015 rpy=0 0 0 -> xyz=-0 0.07 0.015 rpy=0 0 0
- joint right_finger2_j2: origin xyz=-0 0.01 -0 rpy=0 1.5708 0 -> xyz=0 0.01 -0 rpy=-0 1.5708 0
- joint right_finger2_j3: origin xyz=0 0.03 0 rpy=0 -1.5708 0 -> xyz=0 0.03 -0 rpy=0 -1.5708 0
- joint right_finger2_j4: origin xyz=0 0.025 -0 rpy=0 0 0 -> xyz=0 0.025 0 rpy=0 -0 -0
- joint right_finger3_j1: origin xyz=0 0.07 -0 rpy=0 0 -0 -> xyz=0 0.07 -0 rpy=0 0 0
- joint right_finger3_j2: origin xyz=0 0.01 0 rpy=-0 1.5708 0 -> xyz=-0 0.01 0 rpy=0 1.5708 0
- joint right_finger3_j3: origin xyz=0 0.035 0 rpy=0 -1.5708 0 -> xyz=0 0.035 0 rpy=-0 -1.5708 0
- joint right_finger3_j4: origin xyz=-0 0.03 -0 rpy=0 0 0 -> xyz=0 0.03 0 rpy=-0 0 -0
- joint right_finger4_j1: origin xyz=0 0.07 -0.015 rpy=-0 0 -0 -> xyz=0 0.07 -0.015 rpy=0 0 0
- joint right_finger4_j2: origin xyz=0 0.01 0 rpy=-0 1.5708 0 -> xyz=-0 0.01 0 rpy=-0 1.5708 0
- joint right_finger4_j3: origin xyz=0 0.035 -0 rpy=-0 -1.5708 0 -> xyz=0 0.035 -0 rpy=0 -1.5708 0
- joint right_finger4_j4: origin xyz=0 0.025 0 rpy=-0 0 0 -> xyz=0 0.025 -0 rpy=0 0 -0
- joint right_finger5_j1: origin xyz=0 0.07 -0.03 rpy=0 0 -0 -> xyz=0 0.07 -0.03 rpy=0 0 0
- joint right_finger5_j2: origin xyz=0 0.01 -0 rpy=-0 1.5708 0 -> xyz=0 0.01 0 rpy=-0 1.5708 0
- joint right_finger5_j3: origin xyz=0 0.025 -0 rpy=-0 -1.5708 0 -> xyz=-0 0.025 -0 rpy=-0 -1.5708 0
- joint right_finger5_j4: origin xyz=-0 0.02 0 rpy=0 0 0 -> xyz=0 0.02 0 rpy=-0 -0 0
- joint right_hip_pitch: origin xyz=0 -0.08 0 rpy=-1.5708 0 0 -> xyz=1.36e-09 -0.08 -1.6286e-08 rpy=-1.39626 -0 -0
- joint right_hip_roll: origin xyz=-0 -0 0 rpy=0 1.5708 0 -> xyz=-0 0 -0 rpy=-1.5708 1.39626 -1.5708
- joint right_knee_pitch: origin xyz=-0 -0 -0.42 rpy=-1.5708 0 0 -> xyz=0 0 -0.42 rpy=-1.5708 0 -0
- joint right_shoulder_pitch: origin xyz=-0.09 0.17 -0 rpy=-3.14159 -1.5708 0 -> xyz=-0.0887752 0.176946 0 rpy=2.96706 -1.5708 0
- joint right_shoulder_roll: limit lower=-1.74533 upper=1.74533 effort=100 velocity=100 -> lower=-0.174533 upper=3.14159 effort=100 velocity=100; origin xyz=-0 0 0 rpy=1.5708 -0 1.5708 -> xyz=0 -0 0 rpy=1.5708 -0.174533 1.5708
- joint right_wrist_pitch: origin xyz=0 0 0 rpy=0 1.5708 0 -> xyz=0 0 -0 rpy=0 1.5708 0
- joint right_wrist_roll: origin xyz=-0 0 0 rpy=1.5708 0 0 -> xyz=0 0 0 rpy=1.5708 0 0
- joint right_wrist_yaw: origin xyz=0 0.18 0 rpy=-1.5708 -0 -0 -> xyz=0 0.18 0 rpy=-1.5708 0 -0
- joint waist_pitch: origin xyz=0 -0 0 rpy=1.5708 0 3.14159 -> xyz=0 0 0 rpy=1.5708 0 -3.14159
- joint waist_roll: origin xyz=-0 0.09 -0 rpy=0 -1.5708 0 -> xyz=0 0.09 -0 rpy=0 -1.5708 0
- joint waist_yaw: origin xyz=0 -0 0.12 rpy=-0 -0 0 -> xyz=-0 -0 0.12 rpy=0 0 -0

Commit message: fix: shoulder roll limit

File: data/miku/urdf/miku.urdf (robot description, URDF)
Before this commit: robot miku, 75 links, 74 joints
Joints:
- joint left_ankle_pitch: origin xyz=0 0 0 rpy=-0 -1.5708 0 -> xyz=0 0 0 rpy=0 -1.5708 0
- joint left_elbow_pitch: origin xyz=0 -0 0.2 rpy=1.5708 -0 -0 -> xyz=0 -0 0.2 rpy=1.5708 0 -0
- joint left_finger1_j1: origin xyz=-0 0.035 0.015 rpy=0.785398 0 0 -> xyz=0 0.035 0.015 rpy=0.785398 0 -0
- joint left_finger1_j2: origin xyz=0 0.01 -0 rpy=0 -1.5708 0 -> xyz=0 0.01 0 rpy=0 -1.5708 0
- joint left_finger1_j3: origin xyz=-0 0.025 0 rpy=0 1.5708 0 -> xyz=-0 0.025 0 rpy=-0 1.5708 0
- joint left_finger1_j4: origin xyz=0 0.025 0 rpy=0 -0 -0 -> xyz=-0 0.025 0 rpy=-0 0 -0
- joint left_finger2_j1: origin xyz=-0 0.07 0.015 rpy=0 0 -0 -> xyz=0 0.07 0.015 rpy=-0 0 -0
- joint left_finger2_j3: origin xyz=0 0.03 0 rpy=-0 1.5708 0 -> xyz=0 0.03 -0 rpy=0 1.5708 0
- joint left_finger2_j4: origin xyz=0 0.025 -0 rpy=0 0 -0 -> xyz=0 0.025 0 rpy=0 0 0
- joint left_finger3_j1: origin xyz=0 0.07 0 rpy=-0 0 0 -> xyz=-0 0.07 0 rpy=0 -0 -0
- joint left_finger3_j2: origin xyz=0 0.01 0 rpy=0 -1.5708 0 -> xyz=0 0.01 -0 rpy=-0 -1.5708 0
- joint left_finger3_j3: origin xyz=0 0.035 0 rpy=-0 1.5708 0 -> xyz=-0 0.035 0 rpy=-0 1.5708 0
- joint left_finger3_j4: origin xyz=0 0.03 -0 rpy=0 0 -0 -> xyz=0 0.03 -0 rpy=-0 -0 0
- joint left_finger4_j1: origin xyz=0 0.07 -0.015 rpy=-0 0 0 -> xyz=0 0.07 -0.015 rpy=0 -0 -0
- joint left_finger4_j2: origin xyz=0 0.01 0 rpy=0 -1.5708 0 -> xyz=-0 0.01 -0 rpy=0 -1.5708 0
- joint left_finger4_j3: origin xyz=0 0.035 0 rpy=0 1.5708 0 -> xyz=0 0.035 -0 rpy=0 1.5708 0
- joint left_finger5_j1: origin xyz=0 0.07 -0.03 rpy=0 0 0 -> xyz=-0 0.07 -0.03 rpy=0 0 -0
- joint left_finger5_j2: origin xyz=0 0.01 0 rpy=-0 -1.5708 0 -> xyz=-0 0.01 0 rpy=0 -1.5708 0
- joint left_finger5_j3: origin xyz=0 0.025 0 rpy=-0 1.5708 0 -> xyz=0 0.025 0 rpy=0 1.5708 0
- joint left_finger5_j4: origin xyz=0 0.02 0 rpy=-0 -0 0 -> xyz=-0 0.02 0 rpy=-0 -0 0
- joint left_knee_pitch: origin xyz=-0 -0 -0.42 rpy=-1.5708 0 -0 -> xyz=-0 0 -0.42 rpy=-1.5708 0 -0
- joint left_shoulder_roll: limit lower=-0.174533 upper=3.14159 effort=100 velocity=100 -> lower=-1.74533 upper=1.5708 effort=100 velocity=100; origin xyz=-0 0 0 rpy=1.5708 0.174533 1.5708 -> xyz=0 0 0 rpy=1.5708 0.174533 1.5708
- joint left_shoulder_yaw: origin xyz=0 0 0 rpy=-1.5708 -1.5708 0 -> xyz=0 0 -0 rpy=-1.5708 -1.5708 0
- joint left_wrist_pitch: origin xyz=0 0 0 rpy=0 1.5708 0 -> xyz=0 -0 -0 rpy=0 1.5708 0
- joint left_wrist_roll: origin xyz=0 0 0 rpy=1.5708 0 -0 -> xyz=-0 0 0 rpy=1.5708 0 -0
- joint left_wrist_yaw: origin xyz=0 0.18 -0 rpy=-1.5708 -0 0 -> xyz=-0 0.18 0 rpy=-1.5708 -0 0
- joint neck_pitch: origin xyz=0 0.04 0 rpy=-0 1.5708 0 -> xyz=0 0.04 0 rpy=0 1.5708 0
- joint neck_roll: origin xyz=-0 -0 0.04 rpy=1.5708 0 1.5708 -> xyz=0 -0 0.04 rpy=1.5708 -0 1.5708
- joint right_ankle_roll: origin xyz=0 0 0 rpy=-1.5708 0 -1.5708 -> xyz=-0 0 0 rpy=-1.5708 0 -1.5708
- joint right_ankle_yaw: origin xyz=0 0.4 0 rpy=1.5708 -0 -0 -> xyz=-0 0.4 0 rpy=1.5708 -0 -0
- joint right_elbow_pitch: origin xyz=0 0 0.2 rpy=1.5708 0 -0 -> xyz=0 0 0.2 rpy=1.5708 -0 -0
- joint right_finger1_j3: origin xyz=-0 0.025 0 rpy=0 -1.5708 0 -> xyz=0 0.025 -0 rpy=-0 -1.5708 0
- joint right_finger1_j4: origin xyz=0 0.025 0 rpy=-0 0 -0 -> xyz=0 0.025 0 rpy=-0 -0 -0
- joint right_finger2_j1: origin xyz=-0 0.07 0.015 rpy=0 0 0 -> xyz=0 0.07 0.015 rpy=0 0 -0
- joint right_finger2_j2: origin xyz=0 0.01 -0 rpy=-0 1.5708 0 -> xyz=0 0.01 0 rpy=-0 1.5708 0
- joint right_finger2_j3: origin xyz=0 0.03 -0 rpy=0 -1.5708 0 -> xyz=0 0.03 0 rpy=0 -1.5708 0
- joint right_finger3_j1: origin xyz=0 0.07 -0 rpy=0 0 0 -> xyz=-0 0.07 -0 rpy=0 0 0
- joint right_finger3_j2: origin xyz=-0 0.01 0 rpy=0 1.5708 0 -> xyz=0 0.01 0 rpy=0 1.5708 0
- joint right_finger3_j3: origin xyz=0 0.035 0 rpy=-0 -1.5708 0 -> xyz=-0 0.035 0 rpy=0 -1.5708 0
- joint right_finger3_j4: origin xyz=0 0.03 0 rpy=-0 0 -0 -> xyz=0 0.03 0 rpy=-0 -0 -0
- joint right_finger4_j1: origin xyz=0 0.07 -0.015 rpy=0 0 0 -> xyz=0 0.07 -0.015 rpy=0 0 -0
- joint right_finger4_j2: origin xyz=-0 0.01 0 rpy=-0 1.5708 0 -> xyz=-0 0.01 0 rpy=0 1.5708 0
- joint right_finger4_j3: origin xyz=0 0.035 -0 rpy=0 -1.5708 0 -> xyz=0 0.035 0 rpy=-0 -1.5708 0
- joint right_finger4_j4: origin xyz=0 0.025 -0 rpy=0 0 -0 -> xyz=0 0.025 0 rpy=-0 0 -0
- joint right_finger5_j1: origin xyz=0 0.07 -0.03 rpy=0 0 0 -> xyz=0 0.07 -0.03 rpy=0 0 -0
- joint right_finger5_j2: origin xyz=0 0.01 0 rpy=-0 1.5708 0 -> xyz=0 0.01 0 rpy=0 1.5708 0
- joint right_finger5_j4: origin xyz=0 0.02 0 rpy=-0 -0 0 -> xyz=0 0.02 0 rpy=-0 -0 -0
- joint right_hip_pitch: origin xyz=1.36e-09 -0.08 -1.6286e-08 rpy=-1.39626 -0 -0 -> xyz=1.36e-09 -0.08 -1.6286e-08 rpy=-1.39626 -0 0
- joint right_hip_roll: origin xyz=-0 0 -0 rpy=-1.5708 1.39626 -1.5708 -> xyz=-0 0 0 rpy=-1.5708 1.39626 -1.5708
- joint right_knee_pitch: origin xyz=0 0 -0.42 rpy=-1.5708 0 -0 -> xyz=0 -0 -0.42 rpy=-1.5708 0 -0
- joint right_shoulder_roll: limit lower=-0.174533 upper=3.14159 effort=100 velocity=100 -> lower=-1.74533 upper=1.5708 effort=100 velocity=100; origin xyz=0 -0 0 rpy=1.5708 -0.174533 1.5708 -> xyz=-0 0 0 rpy=1.5708 -0.174533 1.5708
- joint right_wrist_pitch: origin xyz=0 0 -0 rpy=0 1.5708 0 -> xyz=0 0 0 rpy=0 1.5708 0
- joint right_wrist_yaw: origin xyz=0 0.18 0 rpy=-1.5708 0 -0 -> xyz=0 0.18 0 rpy=-1.5708 -0 0
- joint waist_pitch: origin xyz=0 0 0 rpy=1.5708 0 -3.14159 -> xyz=-0 0 0 rpy=1.5708 0 3.14159
- joint waist_roll: origin xyz=0 0.09 -0 rpy=0 -1.5708 0 -> xyz=0 0.09 0 rpy=-0 -1.5708 0
- joint waist_yaw: origin xyz=-0 -0 0.12 rpy=0 0 -0 -> xyz=-0 0 0.12 rpy=0 0 0

Commit message: update: correct frame orientations

File: data/miku/urdf/miku.urdf (robot description, URDF)
Before this commit: robot miku, 75 links, 74 joints
Joints:
- joint left_ankle_pitch: origin xyz=0 0 0 rpy=0 -1.5708 0 -> xyz=0 0 0 rpy=-0 -1.5708 0
- joint left_ankle_roll: origin xyz=0 0 0 rpy=-1.5708 -0 -1.5708 -> xyz=0 0 0 rpy=-1.5708 0 -1.5708
- joint left_ankle_yaw: origin xyz=0 0.4 0 rpy=1.5708 -0 0 -> xyz=0 0.4 0 rpy=1.5708 -0 -0
- joint left_elbow_pitch: origin xyz=0 -0 0.2 rpy=1.5708 0 -0 -> xyz=-0 0 -0.2 rpy=-1.5708 0 0
- joint left_finger1_j1: origin xyz=0 0.035 0.015 rpy=0.785398 0 -0 -> xyz=0 0.035 0.015 rpy=0.785398 -0 -0
- joint left_finger1_j3: origin xyz=-0 0.025 0 rpy=-0 1.5708 0 -> xyz=0 0.025 0 rpy=-0 1.5708 0
- joint left_finger1_j4: origin xyz=-0 0.025 0 rpy=-0 0 -0 -> xyz=0 0.025 0 rpy=-0 0 0
- joint left_finger2_j1: origin xyz=0 0.07 0.015 rpy=-0 0 -0 -> xyz=0 0.07 0.015 rpy=-0 -0 -0
- joint left_finger2_j2: origin xyz=-0 0.01 0 rpy=-0 -1.5708 0 -> xyz=0 0.01 -0 rpy=-0 -1.5708 0
- joint left_finger2_j3: origin xyz=0 0.03 -0 rpy=0 1.5708 0 -> xyz=-0 0.03 0 rpy=-0 1.5708 0
- joint left_finger2_j4: origin xyz=0 0.025 0 rpy=0 0 0 -> xyz=0 0.025 0 rpy=-0 0 -0
- joint left_finger3_j1: origin xyz=-0 0.07 0 rpy=0 -0 -0 -> xyz=0 0.07 0 rpy=-0 0 -0
- joint left_finger3_j2: origin xyz=0 0.01 -0 rpy=-0 -1.5708 0 -> xyz=0 0.01 0 rpy=0 -1.5708 0
- joint left_finger3_j3: origin xyz=-0 0.035 0 rpy=-0 1.5708 0 -> xyz=0 0.035 0 rpy=0 1.5708 0
- joint left_finger3_j4: origin xyz=0 0.03 -0 rpy=-0 -0 0 -> xyz=0 0.03 -0 rpy=-0 -0 -0
- joint left_finger4_j1: origin xyz=0 0.07 -0.015 rpy=0 -0 -0 -> xyz=-0 0.07 -0.015 rpy=-0 -0 -0
- joint left_finger4_j2: origin xyz=-0 0.01 -0 rpy=0 -1.5708 0 -> xyz=-0 0.01 0 rpy=0 -1.5708 0
- joint left_finger4_j3: origin xyz=0 0.035 -0 rpy=0 1.5708 0 -> xyz=0 0.035 0 rpy=0 1.5708 0
- joint left_finger4_j4: origin xyz=0 0.025 0 rpy=-0 0 0 -> xyz=0 0.025 0 rpy=-0 0 -0
- joint left_finger5_j1: origin xyz=-0 0.07 -0.03 rpy=0 0 -0 -> xyz=0 0.07 -0.03 rpy=-0 -0 -0
- joint left_finger5_j4: origin xyz=-0 0.02 0 rpy=-0 -0 0 -> xyz=0 0.02 0 rpy=-0 -0 -0
- joint left_hip_pitch: origin xyz=1.36e-09 0.08 1.6286e-08 rpy=-1.74533 0 0 -> xyz=1.36e-09 0.08 1.6286e-08 rpy=-1.74533 0 -0
- joint left_hip_roll: origin xyz=-0 0 -0 rpy=1.5708 1.39626 1.5708 -> xyz=-0 0 0 rpy=1.5708 1.39626 1.5708
- joint left_hip_yaw: origin xyz=-0 0 0 rpy=1.5708 -1.5708 0 -> xyz=0 0 0 rpy=1.5708 -1.5708 0
- joint left_knee_pitch: origin xyz=-0 0 -0.42 rpy=-1.5708 0 -0 -> xyz=0 -0 -0.42 rpy=-1.5708 -0 0
- joint left_shoulder_roll: origin xyz=0 0 0 rpy=1.5708 0.174533 1.5708 -> xyz=0 -0 0 rpy=1.5708 0.174533 1.5708
- joint left_shoulder_yaw: origin xyz=0 0 -0 rpy=-1.5708 -1.5708 0 -> xyz=0 0 -0 rpy=1.5708 -1.5708 0
- joint left_wrist_pitch: origin xyz=0 -0 -0 rpy=0 1.5708 0 -> xyz=0 0 0 rpy=0 1.5708 0
- joint left_wrist_roll: origin xyz=-0 0 0 rpy=1.5708 0 -0 -> xyz=-0 0 0 rpy=-1.5708 0 0
- joint left_wrist_yaw: origin xyz=-0 0.18 0 rpy=-1.5708 -0 0 -> xyz=0 0.18 0 rpy=1.5708 -0 0
- joint neck_pitch: origin xyz=0 0.04 0 rpy=0 1.5708 0 -> xyz=-0 0.04 -0 rpy=0 1.5708 0
- joint right_ankle_pitch: origin xyz=0 0 0 rpy=0 -1.5708 0 -> xyz=0 0 0 rpy=-0 -1.5708 0
- joint right_ankle_roll: origin xyz=-0 0 0 rpy=-1.5708 0 -1.5708 -> xyz=0 0 0 rpy=-1.5708 0 -1.5708
- joint right_ankle_yaw: origin xyz=-0 0.4 0 rpy=1.5708 -0 -0 -> xyz=-0 0.4 -0 rpy=1.5708 0 -0
- joint right_elbow_pitch: origin xyz=0 0 0.2 rpy=1.5708 -0 -0 -> xyz=0 0 -0.2 rpy=-1.5708 0 0
- joint right_finger1_j1: origin xyz=0 0.035 0.015 rpy=0.785398 0 0 -> xyz=0 0.035 0.015 rpy=0.785398 -0 0
- joint right_finger1_j2: origin xyz=0 0.01 -0 rpy=-0 1.5708 0 -> xyz=0 0.01 0 rpy=-0 1.5708 0
- joint right_finger1_j3: origin xyz=0 0.025 -0 rpy=-0 -1.5708 0 -> xyz=0 0.025 0 rpy=-0 -1.5708 0
- joint right_finger1_j4: origin xyz=0 0.025 0 rpy=-0 -0 -0 -> xyz=0 0.025 -0 rpy=-0 0 0
- joint right_finger2_j1: origin xyz=0 0.07 0.015 rpy=0 0 -0 -> xyz=0 0.07 0.015 rpy=-0 -0 -0
- joint right_finger2_j2: origin xyz=0 0.01 0 rpy=-0 1.5708 0 -> xyz=0 0.01 -0 rpy=-0 1.5708 0
- joint right_finger2_j3: origin xyz=0 0.03 0 rpy=0 -1.5708 0 -> xyz=-0 0.03 -0 rpy=-0 -1.5708 0
- joint right_finger2_j4: origin xyz=0 0.025 0 rpy=0 -0 -0 -> xyz=0 0.025 -0 rpy=0 0 0
- joint right_finger3_j1: origin xyz=-0 0.07 -0 rpy=0 0 0 -> xyz=0 0.07 0 rpy=-0 -0 -0
- joint right_finger3_j2: origin xyz=0 0.01 0 rpy=0 1.5708 0 -> xyz=0 0.01 0 rpy=-0 1.5708 0
- joint right_finger3_j3: origin xyz=-0 0.035 0 rpy=0 -1.5708 0 -> xyz=0 0.035 0 rpy=0 -1.5708 0
- joint right_finger4_j1: origin xyz=0 0.07 -0.015 rpy=0 0 -0 -> xyz=0 0.07 -0.015 rpy=-0 0 0
- joint right_finger4_j2: origin xyz=-0 0.01 0 rpy=0 1.5708 0 -> xyz=0 0.01 0 rpy=0 1.5708 0
- joint right_finger4_j3: origin xyz=0 0.035 0 rpy=-0 -1.5708 0 -> xyz=0 0.035 -0 rpy=-0 -1.5708 0
- joint right_finger4_j4: origin xyz=0 0.025 0 rpy=-0 0 -0 -> xyz=0 0.025 0 rpy=0 -0 0
- joint right_finger5_j1: origin xyz=0 0.07 -0.03 rpy=0 0 -0 -> xyz=0 0.07 -0.03 rpy=-0 -0 -0
- joint right_finger5_j3: origin xyz=-0 0.025 -0 rpy=-0 -1.5708 0 -> xyz=0 0.025 0 rpy=-0 -1.5708 0
- joint right_finger5_j4: origin xyz=0 0.02 0 rpy=-0 -0 -0 -> xyz=0 0.02 0 rpy=0 0 0
- joint right_hip_pitch: origin xyz=1.36e-09 -0.08 -1.6286e-08 rpy=-1.39626 -0 0 -> xyz=1.36e-09 -0.08 -1.6286e-08 rpy=-1.39626 0 -0
- joint right_hip_roll: origin xyz=-0 0 0 rpy=-1.5708 1.39626 -1.5708 -> xyz=0 0 0 rpy=-1.5708 1.39626 -1.5708
- joint right_knee_pitch: origin xyz=0 -0 -0.42 rpy=-1.5708 0 -0 -> xyz=0 0 -0.42 rpy=-1.5708 0 -0
- joint right_shoulder_roll: origin xyz=-0 0 0 rpy=1.5708 -0.174533 1.5708 -> xyz=0 -0 -0 rpy=-1.5708 0.174533 -1.5708
- joint right_wrist_pitch: origin xyz=0 0 0 rpy=0 1.5708 0 -> xyz=0 0 0 rpy=-0 1.5708 0
- joint right_wrist_roll: origin xyz=0 0 0 rpy=1.5708 0 0 -> xyz=-0 0 0 rpy=-1.5708 -0 0
- joint right_wrist_yaw: origin xyz=0 0.18 0 rpy=-1.5708 -0 0 -> xyz=0 0.18 0 rpy=1.5708 0 -0
