Commit message: update: assets

File: data/miku/urdf/miku.urdf (robot description, URDF)
Before this commit: robot miku, 75 links, 74 joints
Links:
- removed link torso
- added link chest, mass 3.98764; collision box size=0.08 0.1 0.2; visual mesh filename=../meshes/chest_visual.stl
- link head: mass 4.83041 -> 4.7098
- link left_elbow_pitch: mass 0.304342 -> 0.1; geometry visual mesh filename=../meshes/left_elbow_pitch_visual.stl
- link left_hand: mass 0.028365 -> 0.0692791
- link left_shoulder_pitch: mass 0.311646 -> 0.375
- link left_shoulder_roll: mass 0.455782 -> 0.41; geometry visual mesh filename=../meshes/left_shoulder_roll_visual.stl
- link left_shoulder_yaw: mass 0.175301 -> 0.416; geometry collision cylinder length=0.08 radius=0.03; visual mesh filename=../meshes/left_shoulder_yaw_visual.stl
- link left_wrist_roll: mass 0.0779115 -> 0.25
- link left_wrist_yaw: mass 0.0779115 -> 0.6; geometry collision cylinder length=0.08 radius=0.03; visual mesh filename=../meshes/left_wrist_yaw_visual.stl
- link right_elbow_pitch: mass 0.304342 -> 0.1; geometry visual mesh filename=../meshes/right_elbow_pitch_visual.stl
- link right_hand: mass 0.028365 -> 0.0692787
- link right_shoulder_pitch: mass 0.311646 -> 0.375
- link right_shoulder_roll: mass 0.455782 -> 0.41; geometry visual mesh filename=../meshes/right_shoulder_roll_visual.stl
- link right_shoulder_yaw: mass 0.175301 -> 0.416; geometry collision cylinder length=0.08 radius=0.03; visual mesh filename=../meshes/right_shoulder_yaw_visual.stl
- link right_wrist_roll: mass 0.0779115 -> 0.25
- link right_wrist_yaw: mass 0.0779115 -> 0.6; geometry collision cylinder length=0.08 radius=0.03; visual mesh filename=../meshes/right_wrist_yaw_visual.stl
Joints:
- joint left_ankle_pitch: origin xyz=0 0 0 rpy=-0 -1.5708 0 -> xyz=0 0 -0 rpy=-0 -1.5708 0
- joint left_ankle_roll: origin xyz=0 0 0 rpy=-1.5708 0 -1.5708 -> xyz=0 0 0 rpy=-1.5708 -0 -1.5708
- joint left_ankle_yaw: origin xyz=0 0.4 0 rpy=1.5708 -0 -0 -> xyz=-0 0.4 -0 rpy=1.5708 0 0
- joint left_elbow_pitch: origin xyz=-0 0 -0.2 rpy=-1.5708 0 0 -> xyz=0.01 -0 -0.08 rpy=-1.5708 -0 0
- joint left_finger1_j1: origin xyz=0 0.035 0.015 rpy=0.785398 -0 -0 -> xyz=0 0.035 0.03 rpy=0.785398 -0 0
- joint left_finger1_j2: origin xyz=0 0.01 0 rpy=0 -1.5708 0 -> xyz=0 0.01 0 rpy=-0 -1.5708 0
- joint left_finger1_j4: origin xyz=0 0.025 0 rpy=-0 0 0 -> xyz=0 0.025 -0 rpy=0 0 -0
- joint left_finger2_j1: origin xyz=0 0.07 0.015 rpy=-0 -0 -0 -> xyz=0 0.07 0.015 rpy=0 -0 0
- joint left_finger2_j2: origin xyz=0 0.01 -0 rpy=-0 -1.5708 0 -> xyz=0 0.01 0 rpy=-0 -1.5708 0
- joint left_finger2_j3: origin xyz=-0 0.03 0 rpy=-0 1.5708 0 -> xyz=0 0.03 0 rpy=0 1.5708 0
- joint left_finger2_j4: origin xyz=0 0.025 0 rpy=-0 0 -0 -> xyz=0 0.025 0 rpy=0 -0 0
- joint left_finger3_j1: origin xyz=0 0.07 0 rpy=-0 0 -0 -> xyz=0 0.075 0 rpy=0 -0 0
- joint left_finger3_j3: origin xyz=0 0.035 0 rpy=0 1.5708 0 -> xyz=0 0.035 -0 rpy=-0 1.5708 0
- joint left_finger3_j4: origin xyz=0 0.03 -0 rpy=-0 -0 -0 -> xyz=-0 0.03 -0 rpy=0 -0 0
- joint left_finger4_j1: origin xyz=-0 0.07 -0.015 rpy=-0 -0 -0 -> xyz=0 0.07 -0.015 rpy=0 -0 0
- joint left_finger4_j2: origin xyz=-0 0.01 0 rpy=0 -1.5708 0 -> xyz=0 0.01 0 rpy=0 -1.5708 0
- joint left_finger4_j4: origin xyz=0 0.025 0 rpy=-0 0 -0 -> xyz=-0 0.025 -0 rpy=0 -0 0
- joint left_finger5_j1: origin xyz=0 0.07 -0.03 rpy=-0 -0 -0 -> xyz=0 0.065 -0.03 rpy=-0 -0 0
- joint left_finger5_j2: origin xyz=-0 0.01 0 rpy=0 -1.5708 0 -> xyz=0 0.01 0 rpy=0 -1.5708 0
- joint left_finger5_j4: origin xyz=0 0.02 0 rpy=-0 -0 -0 -> xyz=0 0.02 0 rpy=0 -0 0
- joint left_hip_pitch: origin xyz=1.36e-09 0.08 1.6286e-08 rpy=-1.74533 0 -0 -> xyz=1.36e-09 0.08 1.6286e-08 rpy=-1.74533 0 0
- joint left_hip_roll: origin xyz=-0 0 0 rpy=1.5708 1.39626 1.5708 -> xyz=0 0 0 rpy=1.5708 1.39626 1.5708
- joint left_knee_pitch: origin xyz=0 -0 -0.42 rpy=-1.5708 -0 0 -> xyz=-0 0 -0.42 rpy=-1.5708 -0 0
- joint left_shoulder_pitch: origin xyz=0.0887752 0.176946 0 rpy=-2.96706 -1.5708 0 -> xyz=0.09 0.17 0 rpy=-2.96706 -1.5708 0; parent torso -> chest
- joint left_shoulder_roll: limit lower=-1.74533 upper=1.5708 effort=100 velocity=100 -> lower=-1.91986 upper=1.5708 effort=100 velocity=100; origin xyz=0 -0 0 rpy=1.5708 0.174533 1.5708 -> xyz=0 0 0 rpy=1.5708 0.174533 1.5708
- joint left_shoulder_yaw: origin xyz=0 0 -0 rpy=1.5708 -1.5708 0 -> xyz=0 0.12 0 rpy=1.5708 -1.5708 0
- joint left_wrist_pitch: limit lower=-1.5708 upper=1.5708 effort=100 velocity=100 -> lower=-0.785398 upper=0.785398 effort=100 velocity=100; origin xyz=0 0 0 rpy=0 1.5708 0 -> xyz=0 0 0 rpy=-0 1.5708 0
- joint left_wrist_roll: limit lower=-0.349066 upper=0.349066 effort=100 velocity=100 -> lower=-0.698132 upper=0.698132 effort=100 velocity=100; origin xyz=-0 0 0 rpy=-1.5708 0 0 -> xyz=0 0 -0.14 rpy=-1.5708 -0 -0
- joint left_wrist_yaw: origin xyz=0 0.18 0 rpy=1.5708 -0 0 -> xyz=-0.01 0.06 -0 rpy=1.5708 0 0
- joint neck_pitch: origin xyz=-0 0.04 -0 rpy=0 1.5708 0 -> xyz=0 0.04 0 rpy=0 1.5708 0
- joint neck_yaw: origin xyz=-0 0.23 0 rpy=-1.5708 -1.5708 0 -> xyz=-0 0.23 -0.01 rpy=-1.5708 -1.5708 0; parent torso -> chest
- joint right_ankle_pitch: origin xyz=0 0 0 rpy=-0 -1.5708 0 -> xyz=0 -0 0 rpy=0 -1.5708 0
- joint right_ankle_roll: origin xyz=0 0 0 rpy=-1.5708 0 -1.5708 -> xyz=-0 0 -0 rpy=-1.5708 -0 -1.5708
- joint right_ankle_yaw: origin xyz=-0 0.4 -0 rpy=1.5708 0 -0 -> xyz=0 0.4 0 rpy=1.5708 0 -0
- joint right_elbow_pitch: origin xyz=0 0 -0.2 rpy=-1.5708 0 0 -> xyz=0.01 0 -0.08 rpy=-1.5708 -0 -0
- joint right_finger1_j1: origin xyz=0 0.035 0.015 rpy=0.785398 -0 0 -> xyz=0 0.035 0.03 rpy=0.785398 0 -0
- joint right_finger1_j2: origin xyz=0 0.01 0 rpy=-0 1.5708 0 -> xyz=-0 0.01 0 rpy=0 1.5708 0
- joint right_finger1_j3: origin xyz=0 0.025 0 rpy=-0 -1.5708 0 -> xyz=-0 0.025 0 rpy=-0 -1.5708 0
- joint right_finger1_j4: origin xyz=0 0.025 -0 rpy=-0 0 0 -> xyz=0 0.025 -0 rpy=0 0 0
- joint right_finger2_j1: origin xyz=0 0.07 0.015 rpy=-0 -0 -0 -> xyz=0 0.07 0.015 rpy=0 0 -0
- joint right_finger2_j2: origin xyz=0 0.01 -0 rpy=-0 1.5708 0 -> xyz=-0 0.01 0 rpy=-0 1.5708 0
- joint right_finger2_j3: origin xyz=-0 0.03 -0 rpy=-0 -1.5708 0 -> xyz=0 0.03 0 rpy=-0 -1.5708 0
- joint right_finger2_j4: origin xyz=0 0.025 -0 rpy=0 0 0 -> xyz=0 0.025 0 rpy=-0 -0 0
- joint right_finger3_j1: origin xyz=0 0.07 0 rpy=-0 -0 -0 -> xyz=0 0.075 0 rpy=0 0 -0
- joint right_finger3_j2: origin xyz=0 0.01 0 rpy=-0 1.5708 0 -> xyz=-0 0.01 -0 rpy=-0 1.5708 0
- joint right_finger3_j3: origin xyz=0 0.035 0 rpy=0 -1.5708 0 -> xyz=-0 0.035 0 rpy=-0 -1.5708 0
- joint right_finger3_j4: origin xyz=0 0.03 0 rpy=-0 -0 -0 -> xyz=-0 0.03 -0 rpy=0 -0 -0
- joint right_finger4_j1: origin xyz=0 0.07 -0.015 rpy=-0 0 0 -> xyz=0 0.07 -0.015 rpy=0 0 -0
- joint right_finger4_j2: origin xyz=0 0.01 0 rpy=0 1.5708 0 -> xyz=-0 0.01 0 rpy=-0 1.5708 0
- joint right_finger4_j3: origin xyz=0 0.035 -0 rpy=-0 -1.5708 0 -> xyz=0 0.035 0 rpy=0 -1.5708 0
- joint right_finger4_j4: origin xyz=0 0.025 0 rpy=0 -0 0 -> xyz=-0 0.025 -0 rpy=-0 0 0
- joint right_finger5_j1: origin xyz=0 0.07 -0.03 rpy=-0 -0 -0 -> xyz=-0 0.065 -0.03 rpy=0 0 -0
- joint right_finger5_j2: origin xyz=0 0.01 0 rpy=0 1.5708 0 -> xyz=0 0.01 0 rpy=-0 1.5708 0
- joint right_finger5_j3: origin xyz=0 0.025 0 rpy=-0 -1.5708 0 -> xyz=0 0.025 0 rpy=0 -1.5708 0
- joint right_finger5_j4: origin xyz=0 0.02 0 rpy=0 0 0 -> xyz=0 0.02 0 rpy=-0 0 0
- joint right_knee_pitch: origin xyz=0 0 -0.42 rpy=-1.5708 0 -0 -> xyz=0 -0 -0.42 rpy=-1.5708 -0 0
- joint right_shoulder_pitch: origin xyz=-0.0887752 0.176946 0 rpy=2.96706 -1.5708 0 -> xyz=-0.09 0.17 0 rpy=2.96706 -1.5708 0; parent torso -> chest
- joint right_shoulder_roll: limit lower=-1.74533 upper=1.5708 effort=100 velocity=100 -> lower=-1.91986 upper=1.5708 effort=100 velocity=100; origin xyz=0 -0 -0 rpy=-1.5708 0.174533 -1.5708 -> xyz=0 0 -0 rpy=-1.5708 0.174533 -1.5708
- joint right_shoulder_yaw: origin xyz=0 0 0 rpy=1.5708 -1.5708 0 -> xyz=-0 0.12 -0 rpy=1.5708 -1.5708 0
- joint right_wrist_pitch: limit lower=-1.5708 upper=1.5708 effort=100 velocity=100 -> lower=-0.785398 upper=0.785398 effort=100 velocity=100; origin xyz=0 0 0 rpy=-0 1.5708 0 -> xyz=0 0 -0 rpy=0 1.5708 0
- joint right_wrist_roll: limit lower=-0.349066 upper=0.349066 effort=100 velocity=100 -> lower=-0.698132 upper=0.698132 effort=100 velocity=100; origin xyz=-0 0 0 rpy=-1.5708 -0 0 -> xyz=0 0 -0.14 rpy=-1.5708 0 0
- joint right_wrist_yaw: origin xyz=0 0.18 0 rpy=1.5708 0 -0 -> xyz=-0.01 0.06 -0 rpy=1.5708 -0 0
- joint waist_pitch: origin xyz=-0 0 0 rpy=1.5708 0 3.14159 -> xyz=0 0 0 rpy=1.5708 0 -3.14159
- joint waist_roll: child torso -> chest; origin xyz=0 0.09 0 rpy=-0 -1.5708 0 -> xyz=0 0.09 -0 rpy=0 -1.5708 0
- joint waist_yaw: origin xyz=-0 0 0.12 rpy=0 0 0 -> xyz=0 -0 0.12 rpy=-0 -0 -0
