Commit message: fix: urdf colliders

File: robots/lite/urdf/lite.urdf (robot description, URDF)
Before this commit: robot lite, 75 links, 74 joints
Links:
- link chest: geometry collision box size=0.08 0.1 0.18; visual mesh filename=../meshes/chest_visual.stl
- link left_foot: geometry collision box size=0.065 0.12 0.03; collision box size=0.07 0.05 0.03
- link left_hip_roll: geometry collision cylinder length=0.15 radius=0.05; visual mesh filename=../meshes/left_hip_roll_visual.stl
- link left_knee_pitch: geometry collision cylinder length=0.16 radius=0.045; visual mesh filename=../meshes/left_knee_pitch_visual.stl
- link left_wrist_yaw: geometry collision cylinder length=0.06 radius=0.03; visual mesh filename=../meshes/left_wrist_yaw_visual.stl
- link pelvis: geometry collision cylinder length=0.16 radius=0.05; visual mesh filename=../meshes/pelvis_visual.stl
- link right_foot: geometry collision box size=0.065 0.12 0.03; collision box size=0.07 0.05 0.03
- link right_hip_roll: geometry collision cylinder length=0.15 radius=0.05; visual mesh filename=../meshes/right_hip_roll_visual.stl
- link right_knee_pitch: geometry collision cylinder length=0.16 radius=0.045; visual mesh filename=../meshes/right_knee_pitch_visual.stl
- link right_wrist_yaw: geometry collision cylinder length=0.06 radius=0.03; visual mesh filename=../meshes/right_wrist_yaw_visual.stl
Joints:
- joint left_finger1_j1: origin xyz=0 0.035 0.03 rpy=0.785398 -0 0 -> xyz=0 0.035 0.03 rpy=0.785398 -0 -0
- joint left_finger1_j2: origin xyz=0 0.01 0 rpy=0 -1.5708 0 -> xyz=0 0.01 0 rpy=-0 -1.5708 0
- joint left_finger1_j4: origin xyz=0 0.025 -0 rpy=-0 0 -0 -> xyz=0 0.025 0 rpy=-0 0 -0
- joint left_finger2_j1: origin xyz=0 0.07 0.015 rpy=-0 0 0 -> xyz=-0 0.07 0.015 rpy=-0 0 0
- joint left_finger2_j2: origin xyz=0 0.01 0 rpy=0 -1.5708 0 -> xyz=-0 0.01 -0 rpy=-0 -1.5708 0
- joint left_finger2_j3: origin xyz=0 0.03 0 rpy=-0 1.5708 0 -> xyz=0 0.03 -0 rpy=-0 1.5708 0
- joint left_finger2_j4: origin xyz=0 0.025 0 rpy=-0 0 -0 -> xyz=0 0.025 0 rpy=-0 -0 0
- joint left_finger3_j2: origin xyz=-0 0.01 0 rpy=0 -1.5708 0 -> xyz=-0 0.01 -0 rpy=0 -1.5708 0
- joint left_finger3_j3: origin xyz=-0 0.035 0 rpy=0 1.5708 0 -> xyz=0 0.035 -0 rpy=-0 1.5708 0
- joint left_finger3_j4: origin xyz=-0 0.03 0 rpy=-0 0 0 -> xyz=0 0.03 0 rpy=-0 0 0
- joint left_finger4_j1: origin xyz=-0 0.07 -0.015 rpy=-0 0 0 -> xyz=0 0.07 -0.015 rpy=-0 0 0
- joint left_finger4_j2: origin xyz=-0 0.01 0 rpy=0 -1.5708 0 -> xyz=0 0.01 -0 rpy=0 -1.5708 0
- joint left_finger4_j3: origin xyz=-0 0.035 0 rpy=-0 1.5708 0 -> xyz=0 0.035 0 rpy=-0 1.5708 0
- joint left_finger4_j4: origin xyz=0 0.025 0 rpy=0 -0 -0 -> xyz=0 0.025 -0 rpy=0 -0 0
- joint left_finger5_j2: origin xyz=0 0.01 -0 rpy=0 -1.5708 0 -> xyz=0 0.01 0 rpy=-0 -1.5708 0
- joint left_finger5_j3: origin xyz=0 0.025 0 rpy=0 1.5708 0 -> xyz=-0 0.025 0 rpy=0 1.5708 0
- joint left_finger5_j4: origin xyz=0 0.02 0 rpy=-0 -0 -0 -> xyz=-0 0.02 -0 rpy=-0 -0 0
- joint left_shoulder_yaw: origin xyz=-0 0.12 0 rpy=1.5708 -1.5708 0 -> xyz=-0 0.12 -0 rpy=1.5708 -1.5708 0
- joint left_wrist_roll: origin xyz=0 0 -0.135 rpy=-1.5708 0 -0 -> xyz=0 0 -0.135 rpy=-1.5708 -0 0
- joint right_finger1_j1: origin xyz=-0 0.035 0.03 rpy=0.785398 -0 0 -> xyz=0 0.035 0.03 rpy=0.785398 -0 0
- joint right_finger1_j3: origin xyz=-0 0.025 0 rpy=-0 -1.5708 0 -> xyz=0 0.025 0 rpy=0 -1.5708 0
- joint right_finger1_j4: origin xyz=0 0.025 0 rpy=0 0 -0 -> xyz=0 0.025 -0 rpy=-0 0 -0
- joint right_finger2_j1: origin xyz=-0 0.07 0.015 rpy=-0 -0 0 -> xyz=-0 0.07 0.015 rpy=0 0 0
- joint right_finger2_j2: origin xyz=0 0.01 0 rpy=-0 1.5708 0 -> xyz=-0 0.01 0 rpy=-0 1.5708 0
- joint right_finger2_j4: origin xyz=0 0.025 0 rpy=-0 -0 -0 -> xyz=-0 0.025 -0 rpy=-0 0 -0
- joint right_finger3_j1: origin xyz=0 0.075 -0 rpy=-0 -0 0 -> xyz=0 0.075 0 rpy=0 0 0
- joint right_finger3_j2: origin xyz=0 0.01 -0 rpy=-0 1.5708 0 -> xyz=-0 0.01 0 rpy=-0 1.5708 0
- joint right_finger3_j4: origin xyz=0 0.03 -0 rpy=0 -0 0 -> xyz=0 0.03 -0 rpy=0 0 -0
- joint right_finger4_j1: origin xyz=0 0.07 -0.015 rpy=-0 -0 0 -> xyz=0 0.07 -0.015 rpy=0 0 0
- joint right_finger4_j2: origin xyz=0 0.01 0 rpy=-0 1.5708 0 -> xyz=-0 0.01 0 rpy=-0 1.5708 0
- joint right_finger4_j3: origin xyz=0 0.035 0 rpy=-0 -1.5708 0 -> xyz=-0 0.035 0 rpy=0 -1.5708 0
- joint right_finger4_j4: origin xyz=0 0.025 0 rpy=0 -0 -0 -> xyz=-0 0.025 0 rpy=0 -0 0
- joint right_finger5_j1: origin xyz=0 0.065 -0.03 rpy=-0 -0 0 -> xyz=0 0.065 -0.03 rpy=-0 0 0
- joint right_finger5_j2: origin xyz=0 0.01 0 rpy=-0 1.5708 0 -> xyz=-0 0.01 0 rpy=-0 1.5708 0
- joint right_finger5_j3: origin xyz=0 0.025 -0 rpy=-0 -1.5708 0 -> xyz=0 0.025 0 rpy=-0 -1.5708 0
- joint right_finger5_j4: origin xyz=-0 0.02 0 rpy=0 -0 0 -> xyz=0 0.02 0 rpy=0 0 -0
- joint right_wrist_roll: origin xyz=0 0 -0.135 rpy=-1.5708 -0 0 -> xyz=0 0 -0.135 rpy=-1.5708 0 0
