Commit message: update: bump lite model

File: robots/lite_dummy/urdf/lite.urdf (robot description, URDF)
Before this commit: robot lite, 20 links, 19 joints
Links:
- link left_elbow_pitch: mass 0.1 -> 0.11
- link left_hand: mass 0.161493 -> 0.167493
- link left_shoulder_roll: mass 0.41 -> 0.42
- link left_shoulder_yaw: mass 0.416 -> 0.43
- link left_wrist_yaw: mass 0.6 -> 0.54
- link right_elbow_pitch: mass 0.1 -> 0.11
- link right_hand: mass 0.161493 -> 0.167493
- link right_shoulder_roll: mass 0.41073 -> 0.42073
- link right_shoulder_yaw: mass 0.416 -> 0.43
- link right_wrist_yaw: mass 0.6 -> 0.54
Joints:
- joint left_wrist_roll: origin xyz=-0 -0 -0.135 rpy=-1.5708 -0 0 -> xyz=0 -0 -0.135 rpy=-1.5708 -0 0
- joint right_wrist_pitch: origin xyz=-0 0 0 rpy=-0 1.5708 0 -> xyz=0 0 0 rpy=-0 1.5708 0
- joint right_wrist_roll: origin xyz=0 0 -0.135 rpy=-1.5708 0 0 -> xyz=-0 0 -0.135 rpy=-1.5708 0 0

Commit message: fix: actuator parameters and colliders

File: robots/lite_dummy/urdf/lite.urdf (robot description, URDF)
Before this commit: robot lite, 20 links, 19 joints
Links:
- link chest: geometry collision box size=0.04 0.08 0.18; collision box size=0.04 0.08 0.18
- link left_hand: geometry collision cylinder length=0.04 radius=0.035; collision cylinder length=0.06 radius=0.006
- link left_shoulder_yaw: geometry collision cylinder length=0.12 radius=0.035; visual mesh filename=../meshes/left_shoulder_yaw_visual.stl
- link left_wrist_yaw: geometry collision cylinder length=0.19 radius=0.03; visual mesh filename=../meshes/left_wrist_yaw_visual.stl
- link right_hand: geometry collision cylinder length=0.04 radius=0.035; collision cylinder length=0.06 radius=0.006
- link right_shoulder_yaw: geometry collision cylinder length=0.12 radius=0.035; visual mesh filename=../meshes/right_shoulder_yaw_visual.stl
- link right_wrist_yaw: geometry collision cylinder length=0.19 radius=0.03; visual mesh filename=../meshes/right_wrist_yaw_visual.stl
Joints:
- joint left_elbow_pitch: origin xyz=0.01 -0 -0.08 rpy=-1.5708 -0 -0 -> xyz=0.01 0 -0.08 rpy=-1.5708 0 0
- joint left_shoulder_pitch: origin xyz=0 0.09 0.39 rpy=-1.39626 -0 -0 -> xyz=0 0.09 0.39 rpy=-1.39626 0 -0
- joint left_shoulder_roll: origin xyz=0 0 -0 rpy=1.5708 0.174533 1.5708 -> xyz=-0 -0 0 rpy=1.5708 0.174533 1.5708
- joint left_shoulder_yaw: origin xyz=0 0.12 -0 rpy=1.5708 -1.5708 0 -> xyz=0 0.12 0 rpy=1.5708 -1.5708 0
- joint left_wrist_pitch: origin xyz=-0 0 0 rpy=0 1.5708 0 -> xyz=-0 0 -0 rpy=0 1.5708 0
- joint left_wrist_roll: origin xyz=0 -0 -0.135 rpy=-1.5708 -0 0 -> xyz=-0 0 -0.135 rpy=-1.5708 0 -0
- joint left_wrist_yaw: origin xyz=-0.01 0.055 0 rpy=1.5708 -0 -0 -> xyz=-0.01 0.055 0 rpy=1.5708 0 -0
- joint right_wrist_pitch: origin xyz=0 0 0 rpy=-0 1.5708 0 -> xyz=-0 -0 -0 rpy=0 1.5708 0
- joint right_wrist_yaw: origin xyz=-0.01 0.055 -0 rpy=1.5708 0 -0 -> xyz=-0.01 0.055 -0 rpy=1.5708 0 0
